File: kicad/External-parts/External-parts.kicad_sch (KiCad schematic)
At the start: 2 parts, among them M1 Motor_DC, U1 TB6612FNG

Commit message: add ultrasonic, speaker, nhd
Other:
- added sheet HC-SR04 Array (ultrasonic.kicad_sch)
- added sheet NHD-0440AZ (nhd_0440az.kicad_sch)
- added sheet Speaker (speaker.kicad_sch)
- company: (none) -> ECE 47700 Team 01
- title: (none) -> Offboard 8-Ohm Speaker
Changed lines of the file:
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@@
 	(generator "eeschema")
 	(generator_version "8.0")
-	(paper "A4")
+	(paper "User" 177.8 127)
+	(title_block
+		(title "Offboard 8-Ohm Speaker")
+		(company "ECE 47700 Team 01")
+	)
 	(wire
 		(pts
@@
 	)
 	(sheet
+		(at 205.74 -62.23)
+		(size 82.55 52.07)
+		(fields_autoplaced yes)
+		(stroke
+			(width 0.1524)
+			(type solid)
+		)
+		(fill
+			(color 0 0 0 0.0000)
+		)
+		(property "Sheetname" "Speaker"
+			(at 205.74 -62.9416 0)
+			(show_name yes)
+			(effects
+				(font
+					(size 1.27 1.27)
+				)
+				(justify left bottom)
+			)
+		)
+		(property "Sheetfile" "speaker.kicad_sch"
+			(at 205.74 -9.5754 0)
+			(show_name yes)
+			(effects
+				(font
+					(size 1.27 1.27)
+				)
+				(justify left top)
+			)
+		)
+		(instances
+			(project "External-parts"
+				(path "/f30e32cb-2739-4c2d-b8a9-29b638d16cbf"
+					(page "6")
+				)
+			)
+		)
+	)
+	(sheet
+		(at -125.73 -74.93)
+		(size 127 67.31)
+		(fields_autoplaced yes)
+		(stroke
+			(width 0.1524)
+			(type solid)
+		)
+		(fill
+			(color 0 0 0 0.0000)
+		)
+		(property "Sheetname" "NHD-0440AZ"
+			(at -125.73 -75.6416 0)
+			(effects
+				(font
+					(size 1.27 1.27)
+				)
+				(justify left bottom)
+			)
+		)
+		(property "Sheetfile" "nhd_0440az.kicad_sch"
+			(at -125.73 -7.0354 0)
+			(effects
+				(font
+					(size 1.27 1.27)
+				)
+				(justify left top)
+			)
+		)
+		(instances
+			(project "External-parts"
+				(path "/f30e32cb-2739-4c2d-b8a9-29b638d16cbf"
+					(page "4")
+				)
+			)
+		)
+	)
+	(sheet
 		(at -128.27 0)
 		(size 128.27 127)
@@
 				)
 			)
+		)
+	)
+	(sheet
+		(at 41.91 -66.04)
+		(size 129.54 53.34)
+		(fields_autoplaced yes)
+		(stroke
+			(width 0.1524)
+			(type solid)
+		)
+		(fill
+			(color 0 0 0 0.0000)
+		)
+		(property "Sheetname" "HC-SR04 Array"
+			(at 41.91 -66.7516 0)
+			(effects
+				(font
+					(size 1.27 1.27)
+				)
+				(justify left bottom)
+			)
+		)
+		(property "Sheetfile" "ultrasonic.kicad_sch"
+			(at 41.91 -12.1154 0)
+			(effects
+				(font
+					(size 1.27 1.27)
+				)
+				(justify left top)
+			)
+		)
+		(instances
+			(project "External-parts"
+				(path "/f30e32cb-2739-4c2d-b8a9-29b638d16cbf"
+					(page "5")
+				)
+			)
